File: schematics/remoteSwitch/remoteSwitch.sch (KiCad schematic (older format))
At the start: 23 parts, among them J1 Conn_01x02, J2 Programmer, J3 Conn_01x02, J4 Conn_01x02, K1 FINDER-40.11, K2 FINDER-40.11, SW1 SW_Push_LED, SW2 SW_Push_LED, SW3 SW_SPST, U1 NRF24L01+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

Commit message: Add mosfets and LEDs to relays
Parts:
- removed D1: B120-E3, Diode_SMD:D_SMA, symbol Diode:B120-E3
- removed J4: Conn_01x02, Connectors_Molex:Molex_MegaFit_2x01x5.70mm_Straight, symbol Connector:Screw_Terminal_01x02
- removed K2: FINDER-40.11, Relay_THT:Relay_SPDT_Finder_40.11, symbol Relay:FINDER-40.11
- added D? (x2): LED, symbol Device:LED
- added D?: B120-E3, Diode_SMD:D_SMA, symbol Diode:B120-E3
- added J?: Conn_01x02, Connectors_Molex:Molex_MegaFit_2x01x5.70mm_Straight, symbol Connector:Screw_Terminal_01x02
- added K?: SRD-03VDC-SL-C, Relay_THT:Relay_SPDT_Finder_40.11, symbol Relay:FINDER-40.11
- added Q? (x2): BSS138, symbol Device:Q_NMOS_GDS
- added R? (x4): R_US, symbol Device:R_US
- K1: value FINDER-40.11 -> SRD-03VDC-SL-C
Connections:
- net labels added: CE1, Relay1, Relay2
- wire segments 99 -> 119
Other:
- note added: "Power"
- note removed: "Power Supply"
- note removed: "TODO: Add transistor or mosfet or something"

Commit message: jumpers for optional pwm control of sw_leds
Parts:
- added JP? (x2): LED_SW1 JPR, symbol Jumper:SolderJumper_3_Bridged12
- D1, D3: renamed from D?; footprint (none) -> LEDs:LED_0603_HandSoldering
- D2: value B120-E3 -> RB060M-60TR
- D4: renamed from D?; value B120-E3 -> RB060M-60TR
- R3: value 4.7k -> 10k
- R4, R5: renamed from R?; value R_US -> 4.7k
- R6, R7: renamed from R?; value R_US -> 470
- gave numbers to parts that had none: 4
Connections:
- net labels added: LED_SW1, LED_SW2
- wire segments 119 -> 120
- no-connect marks 17 -> 15

Commit message: Switches to interrupt and other schematic updates
Parts:
- removed JP? (x2): LED_SW1 JPR, symbol Jumper:SolderJumper_3_Bridged12
- added JP1, JP2: SolderJumper_3_Open, symbol Jumper:SolderJumper_3_Open
- J1: value Conn_01x02 -> Conn_AC_MAINS
- K1, K2: footprint Relay_THT:Relay_SPDT_Finder_40.11 -> Relays_THT:Relay_SPDT_SANYOU_SRD_Series_Form_C
- Q1, Q2: footprint (none) -> TO_SOT_Packages_SMD:SOT-23
- R4, R5, R6, R7: footprint (none) -> Resistors_SMD:R_0805_HandSoldering
- U1: footprint RF_Modules:nRF24L01_Breakout -> remoteSwitch_footprints:NRF24L01_SMD
- U3: footprint SMD_Packages:SOJ-32 -> Housings_DFN_QFN:QFN-32-1EP_4x4mm_Pitch0.4mm
Connections:
- net labels removed: CE, Relay1, Relay2
Changed lines of the file:
@@
 encoding utf-8
 Sheet 1 1
-Title ""
+Title "2 Channel Remote Switch"
 Date ""
-Rev ""
+Rev "0.1"
 Comp ""
-Comment1 ""
-Comment2 ""
-Comment3 ""
-Comment4 ""
+Comment1 "for software control."
+Comment2 "Default LED configuration is always off, bridge to GND for always on, or bridgt to SW_LEDn "
+Comment3 "Accepts inputs from 2 LED arcade buttons and standard light switch"
+Comment4 "Acts as receiver or transmitter for remote switching of AC Mains voltage up to 10 amps"
 $EndDescr
 $Comp
@@
 U 1 1 5B5E5DB0
 P 2200 1300
-F 0 "U2" H 2200 1697 60  0000 C CNN
-F 1 "TSP-03" H 2200 1591 60  0000 C CNN
+F 0 "U2" H 2200 1300 60  0000 C CNN
+F 1 "TSP-03" H 2200 1550 60  0000 C CNN
 F 2 "Connectors_JST:JST_SH_BM04B-SRSS-TB_04x1.00mm_Straight" H 2200 1300 60  0001 C CNN
 F 3 "" H 2200 1300 60  0000 C CNN
@@
 P 850 1350
 F 0 "J1" H 770 1025 50  0000 C CNN
-F 1 "Conn_01x02" H 800 1100 50  0000 C CNN
+F 1 "Conn_AC_MAINS" H 800 1100 50  0000 C CNN
 F 2 "Connectors:PINHEAD1-2" H 850 1350 50  0001 C CNN
 F 3 "~" H 850 1350 50  0001 C CNN
@@
 F 0 "K1" V 9950 1650 50  0000 L CNN
 F 1 "SRD-03VDC-SL-C" V 10050 1400 50  0000 L CNN
-F 2 "Relay_THT:Relay_SPDT_Finder_40.11" H 10590 1660 50  0001 C CNN
+F 2 "Relays_THT:Relay_SPDT_SANYOU_SRD_Series_Form_C" H 10590 1660 50  0001 C CNN
 F 3 "https://www.finder-relais.net/de/finder-relais-serie-40.pdf" H 9450 1700 50  0001 C CNN
 	1    9450 1700
@@
 U 1 1 5B5E6ED7
 P 5000 3350
-F 0 "U3" V 5200 1850 50  0000 R CNN
-F 1 "ATmega328PB-AU" V 4700 1850 50  0000 R CNN
-F 2 "SMD_Packages:SOJ-32" H 5000 3350 50  0001 C CIN
+F 0 "U3" H 5000 3400 50  0000 R CNN
+F 1 "ATmega328PB-AU" H 5750 1900 50  0000 R CNN
+F 2 "Housings_DFN_QFN:QFN-32-1EP_4x4mm_Pitch0.4mm" H 5000 3350 50  0001 C CIN
 F 3 "http://ww1.microchip.com/downloads/en/DeviceDoc/40001906C.pdf" H 5000 3350 50  0001 C CNN
 	1    5000 3350
@@
 	5600 3050 5850 3050
 Wire Wire Line
-	4400 4150 4100 4150
-Wire Wire Line
 	5600 3150 5850 3150
 Wire Wire Line
-	4400 4050 4100 4050
-Wire Wire Line
 	5600 2550 5850 2550
 Wire Wire Line
@@
 Wire Wire Line
 	6300 3650 5600 3650
-Wire Wire Line
-	6300 3650 6500 3650
 Connection ~ 6300 3650
 $Comp
@@
 U 1 1 5B61853C
 P 2300 6300
-F 0 "U1" H 2100 6800 50  0000 C CNN
-F 1 "NRF24L01+" H 1950 6700 50  0000 C CNN
-F 2 "RF_Modules:nRF24L01_Breakout" H 2300 6300 50  0001 C CNN
+F 0 "U1" H 2300 6350 50  0000 C CNN
+F 1 "NRF24L01+" H 2550 5900 50  0000 C CNN
+F 2 "remoteSwitch_footprints:NRF24L01_SMD" H 2300 6300 50  0001 C CNN
 F 3 "" H 2300 6300 50  0001 C CNN
 	1    2300 6300
@@
 U 1 1 5B618BCE
 P 2000 5450
-F 0 "C1" H 2115 5496 50  0000 L CNN
-F 1 "0.1uF" H 2115 5405 50  0000 L CNN
+F 0 "C1" H 1750 5500 50  0000 L CNN
+F 1 "0.1uF" H 1650 5400 50  0000 L CNN
 F 2 "Capacitors_SMD:C_1210_HandSoldering" H 2038 5300 50  0001 C CNN
 F 3 "~" H 2000 5450 50  0001 C CNN
@@
 	8600 2100 8600 1850
 Wire Wire Line
-	5600 4550 5850 4550
-Wire Wire Line
-	5600 4450 5850 4450
-Wire Wire Line
 	1600 6200 1850 6200
 Wire Wire Line
 	1600 6300 1850 6300
-Wire Wire Line
-	4400 3950 4100 3950
 $Comp
 L Connector:Screw_Terminal_01x02 J3
@@
 Controller
 Wire Wire Line
-	5850 3850 5600 3850
-Wire Wire Line
-	5600 3950 5850 3950
-Wire Wire Line
 	5850 4050 5600 4050
 NoConn ~ 4400 2150
-NoConn ~ 5600 2150
 NoConn ~ 5600 2750
 NoConn ~ 5600 2850
-NoConn ~ 5600 3250
 NoConn ~ 5600 3350
 NoConn ~ 5600 3450
@@
 NoConn ~ 9550 1400
 Text Label 5900 4450 2    50   ~ 0
-Relay1
+RELAY1
 Text Label 5900 4550 2    50   ~ 0
-Relay2
-Text Label 1650 6200 2    50   ~ 0
-CE
-Text Label 1650 6300 2    50   ~ 0
+RELAY2
+Text Label 1600 6200 0    50   ~ 0
+CE1
+Text Label 1600 6300 0    50   ~ 0
 SS1
-Text Label 3100 6200 2    50   ~ 0
+Text Label 3000 6200 2    50   ~ 0
 SCK1
-Text Label 3100 6300 2    50   ~ 0
+Text Label 3000 6300 2    50   ~ 0
 MOSI1
-Text Label 3100 6400 2    50   ~ 0
+Text Label 3000 6400 2    50   ~ 0
 MISO1
-Text Label 5600 6150 2    50   ~ 0
+Text Label 5400 6150 2    50   ~ 0
 MOSI0
-Text Label 4450 6050 2    50   ~ 0
+Text Label 4450 6050 0    50   ~ 0
 MISO0
-Text Label 4450 6150 2    50   ~ 0
+Text Label 4450 6150 0    50   ~ 0
 SCK0
-Text Label 4450 6250 2    50   ~ 0
+Text Label 4450 6250 0    50   ~ 0
 RESET
 Text Label 2600 4400 2    50   ~ 0
@@
 Text Label 2600 2950 2    50   ~ 0
 SW1
-Text Label 5850 3850 2    50   ~ 0
-SW1
-Text Label 5850 3950 2    50   ~ 0
+Text Label 5850 3250 2    50   ~ 0
 SW2
 Text Label 5850 4050 2    50   ~ 0
@@
 Text Label 5850 3150 2    50   ~ 0
 SCK1
-Text Label 4200 3950 2    50   ~ 0
+Text Label 4150 3950 0    50   ~ 0
 CE1
-Text Label 4200 4050 2    50   ~ 0
+Text Label 4150 4050 0    50   ~ 0
 SS1
-Text Label 4300 4150 2    50   ~ 0
+Text Label 4150 4150 0    50   ~ 0
 MOSI1
 Text Label 5850 2450 2    50   ~ 0
@@
 F 0 "Q1" H 8355 2346 50  0000 L CNN
 F 1 "BSS138" H 8355 2255 50  0000 L CNN
-F 2 "" H 8350 2400 50  0001 C CNN
+F 2 "TO_SOT_Packages_SMD:SOT-23" H 8350 2400 50  0001 C CNN
 F 3 "~" H 8150 2300 50  0001 C CNN
 	1    8150 2300
@@
 Wire Notes Line
 	6950 6500 6950 500
-Wire Wire Line
-	7950 2300 7600 2300
-Text Label 7700 2300 2    50   ~ 0
+Text Label 7650 2300 0    50   ~ 0
 RELAY2
 Wire Wire Line
@@
 F 0 "R4" H 8018 2546 50  0000 L CNN
 F 1 "4.7k" H 8018 2455 50  0000 L CNN
-F 2 "" V 7990 2490 50  0001 C CNN
+F 2 "Resistors_SMD:R_0805_HandSoldering" V 7990 2490 50  0001 C CNN
 F 3 "~" H 7950 2500 50  0001 C CNN
 	1    7950 2500
@@
 Wire Wire Line
 	7950 2350 7950 2300
-Connection ~ 7950 2300
 $Comp
 L Device:R_US R6
@@
 F 0 "R6" H 8318 1546 50  0000 L CNN
 F 1 "470" H 8318 1455 50  0000 L CNN
-F 2 "" V 8290 1490 50  0001 C CNN
+F 2 "Resistors_SMD:R_0805_HandSoldering" V 8290 1490 50  0001 C CNN
 F 3 "~" H 8250 1500 50  0001 C CNN
 	1    8250 1500
@@
 F 0 "K2" V 9950 4200 50  0000 L CNN
 F 1 "SRD-03VDC-SL-C" V 10050 3900 50  0000 L CNN
-F 2 "Relay_THT:Relay_SPDT_Finder_40.11" H 10590 4160 50  0001 C CNN
+F 2 "Relays_THT:Relay_SPDT_SANYOU_SRD_Series_Form_C" H 10590 4160 50  0001 C CNN
 F 3 "https://www.finder-relais.net/de/finder-relais-serie-40.pdf" H 9450 4200 50  0001 C CNN
 	1    9450 4200
@@
 F 0 "Q2" H 8355 4846 50  0000 L CNN
 F 1 "BSS138" H 8355 4755 50  0000 L CNN
-F 2 "" H 8350 4900 50  0001 C CNN
+F 2 "TO_SOT_Packages_SMD:SOT-23" H 8350 4900 50  0001 C CNN
 F 3 "~" H 8150 4800 50  0001 C CNN
 	1    8150 4800
@@
 	1    0    0    -1
 $EndComp
-Wire Wire Line
-	7950 4800 7600 4800
-Text Label 7700 4800 2    50   ~ 0
+Text Label 7650 4800 0    50   ~ 0
 RELAY1
 Wire Wire Line
@@
 F 0 "R5" H 8018 5046 50  0000 L CNN
 F 1 "4.7k" H 8018 4955 50  0000 L CNN
-F 2 "" V 7990 4990 50  0001 C CNN
+F 2 "Resistors_SMD:R_0805_HandSoldering" V 7990 4990 50  0001 C CNN
 F 3 "~" H 7950 5000 50  0001 C CNN
 	1    7950 5000
@@
 Wire Wire Line
 	7950 4850 7950 4800
-Connection ~ 7950 4800
 $Comp
 L Device:R_US R7
@@
 F 0 "R7" H 8318 4046 50  0000 L CNN
 F 1 "470" H 8318 3955 50  0000 L CNN
-F 2 "" V 8290 3990 50  0001 C CNN
+F 2 "Resistors_SMD:R_0805_HandSoldering" V 8290 3990 50  0001 C CNN
 F 3 "~" H 8250 4000 50  0001 C CNN
 	1    8250 4000
@@
 Connection ~ 8250 4600
 $Comp
-L power:+3.3V #PWR?
+L power:+3.3V #PWR0113
 U 1 1 5B702A3F
 P 6300 3350
-F 0 "#PWR?" H 6300 3200 50  0001 C CNN
+F 0 "#PWR0113" H 6300 3200 50  0001 C CNN
 F 1 "+3.3V" H 6315 3523 50  0000 C CNN
 F 2 "" H 6300 3350 50  0001 C CNN
@@
 	1    0    0    -1
 $EndComp
-Wire Wire Line
-	5600 2250 5850 2250
-Wire Wire Line
-	5600 2350 5850 2350
 NoConn ~ 5600 4150
 Text Label 5950 2250 2    50   ~ 0
@@
 Text Label 5950 2350 2    50   ~ 0
 LED_SW2
-$Comp
-L Jumper:SolderJumper_3_Bridged12 JP?
-U 1 1 5B718587
+Wire Wire Line
+	2000 2950 2050 2950
+Wire Wire Line
+	2050 3050 1800 3050
+Wire Wire Line
+	1650 3250 1650 3300
+Text Label 1400 2850 0    50   ~ 0
+LED_SW1
+Wire Wire Line
+	2050 3800 2000 3800
+Wire Wire Line
+	2050 3900 1800 3900
+Wire Wire Line
+	1650 4100 1650 4150
+Text Label 1400 3700 0    50   ~ 0
+LED_SW2
+$Comp
+L Jumper:SolderJumper_3_Open JP2
+U 1 1 5B74373A
+P 1650 3900
+F 0 "JP2" V 1696 3968 50  0000 L CNN
+F 1 "SolderJumper_3_Open" V 1605 3968 50  0000 L CNN
+F 2 "" H 1650 3900 50  0001 C CNN
+F 3 "~" H 1650 3900 50  0001 C CNN
+	1    1650 3900
+	0    -1   -1   0
+$EndComp
+$Comp
+L Jumper:SolderJumper_3_Open JP1
+U 1 1 5B743823
 P 1650 3050
-F 0 "JP?" V 1696 3118 50  0000 L CNN
-F 1 "LED_SW1 JPR" V 1605 3118 50  0000 L CNN
+F 0 "JP1" V 1696 3118 50  0000 L CNN
+F 1 "SolderJumper_3_Open" V 1605 3118 50  0000 L CNN
 F 2 "" H 1650 3050 50  0001 C CNN
 F 3 "~" H 1650 3050 50  0001 C CNN
@@
 $EndComp
 Wire Wire Line
-	2000 2950 2050 2950
-Wire Wire Line
-	2050 3050 1800 3050
-Wire Wire Line
-	1650 3250 1650 3300
-Wire Wire Line
-	1650 2850 1350 2850
-Text Label 1400 2850 2    50   ~ 0
-LED_SW1
-Wire Wire Line
-	2050 3800 2000 3800
-$Comp
-L Jumper:SolderJumper_3_Bridged12 JP?
-U 1 1 5B7349E8
-P 1650 3900
-F 0 "JP?" V 1696 3968 50  0000 L CNN
-F 1 "LED_SW1 JPR" V 1605 3968 50  0000 L CNN
-F 2 "" H 1650 3900 50  0001 C CNN
-F 3 "~" H 1650 3900 50  0001 C CNN
-	1    1650 3900
-	0    -1   -1   0
-$EndComp
-Wire Wire Line
-	2050 3900 1800 3900
-Wire Wire Line
-	1650 4100 1650 4150
-Wire Wire Line
-	1650 3700 1350 3700
-Text Label 1400 3700 2    50   ~ 0
-LED_SW2
+	5600 4450 5900 4450
+Wire Wire Line
+	5600 4550 5900 4550
+Wire Wire Line
+	5600 2250 5950 2250
+Wire Wire Line
+	5600 2350 5950 2350
+Wire Wire Line
+	6300 3650 6550 3650
+Wire Wire Line
+	4400 4150 4150 4150
+Wire Wire Line
+	4400 3950 4150 3950
+Wire Wire Line
+	4150 4050 4400 4050
+Wire Wire Line
+	1400 2850 1650 2850
+Wire Wire Line
+	1650 3700 1400 3700
+Connection ~ 7950 2300
+Wire Wire Line
+	7950 4800 7650 4800
+Connection ~ 7950 4800
+Wire Wire Line
+	7650 2300 7950 2300
+Wire Wire Line
+	5600 2150 5850 2150
+Text Label 5850 2150 2    50   ~ 0
+SW1
+Wire Wire Line
+	5600 3250 5850 3250
+NoConn ~ 5600 3850
+NoConn ~ 5600 3950
 $EndSCHEMATC
